File: prototype/hardware/colalightslk-proto.brd (EAGLE design)
At the start: 50 x 20 mm, 24 parts, among them IC1 OP200D

Commit message: Updated roles desireable to be none micro specific
Parts:
- added X1: (no value), con-yamaichi:USB-A003
- moved R1 73.1 mm to (38.1, 25.4)
- moved U$2 1.27 mm to (1.27, 10.2)
Changed lines of the file:
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@@
 </element>
 <element name="U$1" library="amino" package="TSSOP-20" value="" x="16.51" y="8.89"/>
-<element name="U$2" library="amino" package="MICROUSB-B-PEG" value="FCI-MICROUSB-B-PEG" x="2.54" y="10.16" rot="R270"/>
+<element name="U$2" library="amino" package="MICROUSB-B-PEG" value="FCI-MICROUSB-B-PEG" x="1.27" y="10.16" rot="R270"/>
 <element name="IC1" library="linear" package="SO08" value="OP200D" x="8.89" y="8.89"/>
-<element name="R1" library="rcl" package="R1210" value="" x="-34.29" y="35.56"/>
+<element name="R1" library="rcl" package="R1210" value="" x="38.1" y="25.4"/>
 <element name="L1" library="inductors" package="ED16" value="ED16" x="33.02" y="10.16" rot="MR180"/>
 <element name="U$3" library="amino" package="IPAK" value="NTD4963N" x="24.13" y="5.08" rot="R270"/>
@@
 <element name="U$9" library="amino" package="NRS60XX" value="NRS6028" x="15.24" y="16.51"/>
 <element name="U$6" library="amino" package="SOIC-8-NARROW" value="NTMD4820NR2G" x="7.62" y="16.51" rot="R270"/>
+<element name="X1" library="con-yamaichi" package="USB-A003" value="" x="-1.27" y="10.16" rot="MR90">
+<attribute name="OC_NEWARK" value="unknown" x="-1.27" y="10.16" size="1.778" layer="28" rot="MR90" display="off"/>
+<attribute name="MPN" value="" x="-1.27" y="10.16" size="1.778" layer="28" rot="MR90" display="off"/>
+<attribute name="MF" value="" x="-1.27" y="10.16" size="1.778" layer="28" rot="MR90" display="off"/>
+<attribute name="OC_FARNELL" value="unknown" x="-1.27" y="10.16" size="1.778" layer="28" rot="MR90" display="off"/>
+</element>
 </elements>
 <signals>
