File: prototype/hardware/colalightslk-proto.sch (EAGLE design)
At the start: 24 parts, among them IC1 OP200D

Commit message: Updated roles desireable to be none micro specific
Parts:
- added X1: (no value), con-yamaichi:USB-A003
Changed lines of the file:
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@@
 <part name="U$6" library="amino" deviceset="NTMD4820NR2G" device=""/>
 <part name="GND6" library="supply1" deviceset="GND" device=""/>
+<part name="X1" library="con-yamaichi" deviceset="USB-A003" device=""/>
 </parts>
 <sheets>
@@
 <instance part="U$6" gate="G$1" x="0" y="111.76"/>
 <instance part="GND6" gate="1" x="35.56" y="111.76"/>
+<instance part="X1" gate="G$1" x="-30.48" y="33.02"/>
 </instances>
 <busses>
